File: ESP-Sensors/ESP-Sensors.sch (KiCad schematic (older format))
At the start: 14 parts, among them J1 PROG_CONN, J2 GPIO, J3 CONN_01X05, J4 +5V GND +3.3V, SW1 SW_Push, SW2 SW_Push, U1 ESP-12E

Commit message: started with pcb tracing of esp-sensor
Parts:
- 10K1: footprint (none) -> Potentiometers:Potentiometer_WirePads_Small
- C1, C2: footprint (none) -> Capacitors_SMD:C_0805_HandSoldering
- C3: footprint (none) -> Capacitors_SMD:c_elec_6.3x7.7
- J1, J3: footprint (none) -> Pin_Headers:Pin_Header_Straight_1x05
- J2: footprint (none) -> Pin_Headers:Pin_Header_Straight_1x12
- J4: footprint (none) -> Pin_Headers:Pin_Header_Straight_1x04
- R1, R2, R3: footprint (none) -> Resistors_SMD:R_0805_HandSoldering
- SW1, SW2: footprint (none) -> Buttons_Switches_THT:SW_PUSH_6mm
- U1: footprint (none) -> ESP8266:ESP-12E
Other:
- note added: "2017-03-21"
- note added: "ESP8266-12E sensor print"
- note added: "Optional power regulator, or feed with 3.3V"
Changed lines of the file:
@@
 LIBS:switches
 LIBS:ESP-RS232
-LIBS:ESP-RS232-cache
+LIBS:ESP-Sensors-cache
 EELAYER 25 0
 EELAYER END
@@
 F 0 "J2" H 7550 5150 50  0000 C CNN
 F 1 "GPIO" V 7650 4500 50  0000 C CNN
-F 2 "" H 7550 4500 50  0001 C CNN
+F 2 "Pin_Headers:Pin_Header_Straight_1x12" H 7550 4500 50  0001 C CNN
 F 3 "" H 7550 4500 50  0001 C CNN
 	1    7550 4500
@@
 F 0 "R2" V 2455 1925 50  0000 C CNN
 F 1 "10K" V 2375 1925 50  0000 C CNN
-F 2 "" V 2305 1925 50  0001 C CNN
+F 2 "Resistors_SMD:R_0805_HandSoldering" V 2305 1925 50  0001 C CNN
 F 3 "" H 2375 1925 50  0001 C CNN
 	1    2375 1925
@@
 F 0 "SW1" H 2600 2475 50  0000 L CNN
 F 1 "SW_Push" H 2550 2315 50  0000 C CNN
-F 2 "" H 2550 2575 50  0001 C CNN
+F 2 "Buttons_Switches_THT:SW_PUSH_6mm" H 2550 2575 50  0001 C CNN
 F 3 "" H 2550 2575 50  0001 C CNN
 	1    2550 2375
@@
 F 0 "R1" V 2080 1900 50  0000 C CNN
 F 1 "10K" V 2000 1900 50  0000 C CNN
-F 2 "" V 1930 1900 50  0001 C CNN
+F 2 "Resistors_SMD:R_0805_HandSoldering" V 1930 1900 50  0001 C CNN
 F 3 "" H 2000 1900 50  0001 C CNN
 	1    2000 1900
@@
 F 0 "10K1" V 2850 2350 50  0000 C CNN
 F 1 "POT" V 2925 2350 50  0000 C CNN
-F 2 "" H 3025 2350 50  0001 C CNN
+F 2 "Potentiometers:Potentiometer_WirePads_Small" H 3025 2350 50  0001 C CNN
 F 3 "" H 3025 2350 50  0001 C CNN
 	1    3025 2350
@@
 F 0 "C3" H 10150 2375 50  0000 L CNN
 F 1 "100µF" H 10150 2175 50  0000 L CNN
-F 2 "" H 10163 2125 50  0001 C CNN
+F 2 "Capacitors_SMD:c_elec_6.3x7.7" H 10163 2125 50  0001 C CNN
 F 3 "" H 10125 2275 50  0001 C CNN
 	1    10125 2275
@@
 F 0 "C1" H 2175 2425 50  0000 L CNN
 F 1 "100nF" H 2175 2225 50  0000 L CNN
-F 2 "" H 2188 2175 50  0001 C CNN
+F 2 "Capacitors_SMD:C_0805_HandSoldering" H 2188 2175 50  0001 C CNN
 F 3 "" H 2150 2325 50  0001 C CNN
 	1    2150 2325
@@
 F 0 "R3" V 5755 1475 50  0000 C CNN
 F 1 "10K" V 5675 1475 50  0000 C CNN
-F 2 "" V 5605 1475 50  0001 C CNN
+F 2 "Resistors_SMD:R_0805_HandSoldering" V 5605 1475 50  0001 C CNN
 F 3 "" H 5675 1475 50  0001 C CNN
 	1    5675 1475
@@
 F 0 "SW2" H 5725 2025 50  0000 L CNN
 F 1 "SW_Push" H 5675 1865 50  0000 C CNN
-F 2 "" H 5675 2125 50  0001 C CNN
+F 2 "Buttons_Switches_THT:SW_PUSH_6mm" H 5675 2125 50  0001 C CNN
 F 3 "" H 5675 2125 50  0001 C CNN
 	1    5675 1925
@@
 	5400 3625 6175 3625
 Wire Wire Line
-	7750 3150 8725 3150
-Wire Wire Line
 	7750 3250 7825 3250
 Wire Wire Line
@@
 L VCC #PWR05
 U 1 1 58DCE941
-P 8725 3050
-F 0 "#PWR05" H 8725 2900 50  0001 C CNN
-F 1 "VCC" H 8725 3200 50  0000 C CNN
-F 2 "" H 8725 3050 50  0001 C CNN
-F 3 "" H 8725 3050 50  0001 C CNN
-	1    8725 3050
+P 8375 3050
+F 0 "#PWR05" H 8375 2900 50  0001 C CNN
+F 1 "VCC" H 8375 3200 50  0000 C CNN
+F 2 "" H 8375 3050 50  0001 C CNN
+F 3 "" H 8375 3050 50  0001 C CNN
+	1    8375 3050
 	1    0    0    -1
 $EndComp
@@
 F 0 "J1" H 7550 3650 50  0000 C CNN
 F 1 "PROG_CONN" V 7650 3350 50  0000 C CNN
-F 2 "" H 7550 3350 50  0001 C CNN
+F 2 "Pin_Headers:Pin_Header_Straight_1x05" H 7550 3350 50  0001 C CNN
 F 3 "" H 7550 3350 50  0001 C CNN
 	1    7550 3350
@@
 $EndComp
 Wire Wire Line
-	8725 3150 8725 3050
+	8375 3150 8375 3050
 Wire Wire Line
 	7750 3950 8225 3950
@@
 U 1 1 58DE8BE3
 P 9450 2025
-F 0 "#U07" H 9675 1775 60  0000 C CNN
+F 0 "#U07" H 9675 1775 60  0001 C CNN
 F 1 "HT7333" H 9375 2225 60  0000 C CNN
 F 2 "" H 9400 1925 60  0001 C CNN
@@
 F 0 "C2" H 3550 4050 50  0000 L CNN
 F 1 "100nF" H 3550 3850 50  0000 L CNN
-F 2 "" H 3563 3800 50  0001 C CNN
+F 2 "Capacitors_SMD:C_0805_HandSoldering" H 3563 3800 50  0001 C CNN
 F 3 "" H 3525 3950 50  0001 C CNN
 	1    3525 3950
@@
 F 0 "U1" H 4500 3225 50  0000 C CNN
 F 1 "ESP-12E" H 4500 3425 50  0000 C CNN
-F 2 "" H 4500 3325 50  0001 C CNN
+F 2 "ESP8266:ESP-12E" H 4500 3325 50  0001 C CNN
 F 3 "" H 4500 3325 50  0001 C CNN
 	1    4500 3325
@@
 F 0 "J3" H 7550 6050 50  0000 C CNN
 F 1 "CONN_01X05" V 7650 5750 50  0000 C CNN
-F 2 "" H 7550 5750 50  0001 C CNN
+F 2 "Pin_Headers:Pin_Header_Straight_1x05" H 7550 5750 50  0001 C CNN
 F 3 "" H 7550 5750 50  0001 C CNN
 	1    7550 5750
@@
 F 0 "J4" H 9475 1350 50  0000 C CNN
 F 1 "+5V  GND  +3.3V" V 9575 1100 50  0000 C CNN
-F 2 "" H 9475 1100 50  0001 C CNN
+F 2 "Pin_Headers:Pin_Header_Straight_1x04" H 9475 1100 50  0001 C CNN
 F 3 "" H 9475 1100 50  0001 C CNN
 	1    9475 1100
@@
 $EndComp
 Connection ~ 10125 2050
+Text Notes 7400 7500 0    60   ~ 0
+ESP8266-12E sensor print
+Text Notes 8225 7650 0    60   ~ 0
+2017-03-21
+Wire Notes Line
+	8650 800  8650 3000
+Wire Notes Line
+	8650 3000 10750 3000
+Wire Notes Line
+	10750 3000 10750 800
+Wire Notes Line
+	10750 800  8650 800
+Wire Wire Line
+	7750 3150 8375 3150
+Text Notes 8675 2975 0    60   ~ 0
+Optional power regulator, or feed with 3.3V
 $EndSCHEMATC
