File: ESP-Sensors/ESP-Sensors.sch (KiCad schematic (older format))
At the start: 14 parts, among them J1 PROG_CONN, J2 GPIO, J3 CONN_01X05, J4 +5V GND +3.3V, SW1 SW_Push, SW2 SW_Push, U1 ESP-12E

Commit message: fixed U2 power connection, more traces
Parts:
- added U2: HT7333, TO_SOT_Packages_SMD:SOT89-3_Housing_Handsoldering, symbol HT7333
Connections:
- net labels removed: HT7333
Changed lines of the file:
@@
 LIBS:switches
 LIBS:ESP-RS232
-LIBS:ESP-Sensors-cache
 EELAYER 25 0
 EELAYER END
@@
 $EndComp
 $Comp
-L GND #PWR1
+L GND #PWR01
 U 1 1 58DBDEBB
 P 2375 2750
-F 0 "#PWR1" H 2375 2500 50  0001 C CNN
+F 0 "#PWR01" H 2375 2500 50  0001 C CNN
 F 1 "GND" H 2375 2600 50  0000 C CNN
 F 2 "" H 2375 2750 50  0001 C CNN
@@
 $EndComp
 $Comp
-L GND #PWR8
+L GND #PWR02
 U 1 1 58DBEC21
 P 10125 2575
-F 0 "#PWR8" H 10125 2325 50  0001 C CNN
+F 0 "#PWR02" H 10125 2325 50  0001 C CNN
 F 1 "GND" H 10125 2425 50  0000 C CNN
 F 2 "" H 10125 2575 50  0001 C CNN
@@
 $EndComp
 $Comp
-L GND #PWR6
+L GND #PWR03
 U 1 1 58DBF081
 P 8375 3575
-F 0 "#PWR6" H 8375 3325 50  0001 C CNN
+F 0 "#PWR03" H 8375 3325 50  0001 C CNN
 F 1 "GND" H 8375 3425 50  0000 C CNN
 F 2 "" H 8375 3575 50  0001 C CNN
@@
 $EndComp
 $Comp
-L GND #PWR3
+L GND #PWR04
 U 1 1 58DCB644
 P 5675 2200
-F 0 "#PWR3" H 5675 1950 50  0001 C CNN
+F 0 "#PWR04" H 5675 1950 50  0001 C CNN
 F 1 "GND" H 5675 2050 50  0000 C CNN
 F 2 "" H 5675 2200 50  0001 C CNN
@@
 GPIO_BUS
 $Comp
-L VCC #PWR5
+L VCC #PWR05
 U 1 1 58DCE941
 P 8375 3050
-F 0 "#PWR5" H 8375 2900 50  0001 C CNN
+F 0 "#PWR05" H 8375 2900 50  0001 C CNN
 F 1 "VCC" H 8375 3200 50  0000 C CNN
 F 2 "" H 8375 3050 50  0001 C CNN
@@
 GPIO15
 $Comp
-L GND #PWR4
+L GND #PWR06
 U 1 1 58DCF2D0
 P 5850 3725
-F 0 "#PWR4" H 5850 3475 50  0001 C CNN
+F 0 "#PWR06" H 5850 3475 50  0001 C CNN
 F 1 "GND" H 5850 3575 50  0000 C CNN
 F 2 "" H 5850 3725 50  0001 C CNN
@@
 	9525 1375 9525 1300
 $Comp
-L GND #PWR7
+L GND #PWR07
 U 1 1 58DE8DA8
 P 9475 1375
-F 0 "#PWR7" H 9475 1125 50  0001 C CNN
+F 0 "#PWR07" H 9475 1125 50  0001 C CNN
 F 1 "GND" H 9475 1225 50  0000 C CNN
 F 2 "" H 9475 1375 50  0001 C CNN
@@
 Connection ~ 3525 3725
 $Comp
-L GND #PWR2
+L GND #PWR08
 U 1 1 58DEA3A3
 P 3525 4200
-F 0 "#PWR2" H 3525 3950 50  0001 C CNN
+F 0 "#PWR08" H 3525 3950 50  0001 C CNN
 F 1 "GND" H 3525 4050 50  0000 C CNN
 F 2 "" H 3525 4200 50  0001 C CNN
@@
 Optional power regulator, or feed with 3.3V
 $Comp
-L HT7333 #U1
-U 1 1 58E20754
+L HT7333 U2
+U 1 1 58E21ABC
 P 9450 2050
-F 0 "#U1" H 9725 1825 60  0000 R CNN
+F 0 "U2" H 9725 1825 60  0000 R CNN
 F 1 "HT7333" H 9375 2275 60  0000 C CNN
-F 2 "" H 9400 1975 60  0001 C CNN
+F 2 "TO_SOT_Packages_SMD:SOT89-3_Housing_Handsoldering" H 9400 1975 60  0001 C CNN
 F 3 "" H 9400 1975 60  0001 C CNN
 	1    9450 2050

Commit message: added different trimmer plus deep_sleep jumper header
Parts:
- added J5: DEEP_SLEEP, Pin_Headers:Pin_Header_Straight_1x02, symbol CONN_01X02
- 10K1: footprint Potentiometers:Potentiometer_WirePads_Small -> Potentiometers:Potentiometer_Trimmer_Vishay_T73YP_Horizontal
- J3: value CONN_01X05 -> SPI
- J4: value +5V GND +3.3V -> +3.3V GND +5V
- SW1: value SW_Push -> RESET
- SW2: value SW_Push -> PROG
Connections:
- wire segments 81 -> 86
- no-connect marks 1 -> 0
Other:
- moved on the sheet: 10K1
Changed lines of the file:
@@
 LIBS:switches
 LIBS:ESP-RS232
+LIBS:ESP-Sensors-cache
 EELAYER 25 0
 EELAYER END
@@
 P 2550 2375
 F 0 "SW1" H 2600 2475 50  0000 L CNN
-F 1 "SW_Push" H 2550 2315 50  0000 C CNN
+F 1 "RESET" H 2550 2315 50  0000 C CNN
 F 2 "Buttons_Switches_THT:SW_PUSH_6mm" H 2550 2575 50  0001 C CNN
 F 3 "" H 2550 2575 50  0001 C CNN
@@
 F 0 "10K1" V 2850 2350 50  0000 C CNN
 F 1 "POT" V 2925 2350 50  0000 C CNN
-F 2 "Potentiometers:Potentiometer_WirePads_Small" H 3025 2350 50  0001 C CNN
+F 2 "Potentiometers:Potentiometer_Trimmer_Vishay_T73YP_Horizontal" H 3025 2350 50  0001 C CNN
 F 3 "" H 3025 2350 50  0001 C CNN
 	1    3025 2350
-	1    0    0    -1
+	-1   0    0    1
 $EndComp
 Text Label 3050 2200 0    60   ~ 0
@@
 P 5675 1925
 F 0 "SW2" H 5725 2025 50  0000 L CNN
-F 1 "SW_Push" H 5675 1865 50  0000 C CNN
+F 1 "PROG" H 5675 1865 50  0000 C CNN
 F 2 "Buttons_Switches_THT:SW_PUSH_6mm" H 5675 2125 50  0001 C CNN
 F 3 "" H 5675 2125 50  0001 C CNN
@@
 	2000 3225 3600 3225
 Wire Wire Line
-	3175 2350 3325 2350
-Wire Wire Line
-	3325 2350 3325 3125
-Wire Wire Line
-	3325 3125 3600 3125
+	2825 3125 3600 3125
 Wire Wire Line
 	3025 2650 3025 2500
@@
 	2950 4875 6275 4875
 Wire Wire Line
-	3600 3325 3050 3325
+	2750 3325 3600 3325
 Wire Wire Line
 	3600 3425 3050 3425
@@
 Entry Wire Line
 	3050 3425 2950 3525
-Entry Wire Line
-	3050 3325 2950 3425
 Wire Wire Line
 	3450 3725 3600 3725
@@
 Text Label 3150 3525 0    60   ~ 0
 GPIO12
-NoConn ~ 3600 3325
 Entry Wire Line
 	4550 4775 4650 4875
@@
 P 7550 5750
 F 0 "J3" H 7550 6050 50  0000 C CNN
-F 1 "CONN_01X05" V 7650 5750 50  0000 C CNN
+F 1 "SPI" V 7650 5750 50  0000 C CNN
 F 2 "Pin_Headers:Pin_Header_Straight_1x05" H 7550 5750 50  0001 C CNN
 F 3 "" H 7550 5750 50  0001 C CNN
@@
 P 9475 1100
 F 0 "J4" H 9475 1350 50  0000 C CNN
-F 1 "+5V  GND  +3.3V" V 9575 1100 50  0000 C CNN
+F 1 "+3.3V GND +5V" V 9575 1100 50  0000 C CNN
 F 2 "Pin_Headers:Pin_Header_Straight_1x04" H 9475 1100 50  0001 C CNN
 F 3 "" H 9475 1100 50  0001 C CNN
@@
 	1    0    0    -1
 $EndComp
+$Comp
+L CONN_01X02 J5
+U 1 1 58E29D26
+P 2250 3650
+F 0 "J5" H 2250 3800 50  0000 C CNN
+F 1 "DEEP_SLEEP" V 2350 3650 50  0000 C CNN
+F 2 "Pin_Headers:Pin_Header_Straight_1x02" H 2250 3650 50  0001 C CNN
+F 3 "" H 2250 3650 50  0001 C CNN
+	1    2250 3650
+	-1   0    0    1
+$EndComp
+Wire Wire Line
+	2750 3325 2750 3700
+Wire Wire Line
+	2750 3700 2450 3700
+Wire Wire Line
+	2450 3600 2650 3600
+Wire Wire Line
+	2650 3600 2650 2875
+Wire Wire Line
+	2650 2875 3600 2875
+Connection ~ 3600 2875
+Wire Wire Line
+	2825 3125 2825 2350
+Wire Wire Line
+	2825 2350 2875 2350
 $EndSCHEMATC

Commit message: Added GPIO refs again and added VCC header
Parts:
- J3: footprint Pin_Headers:Pin_Header_Straight_1x05 -> ESP-RS232:SPI_Header
Changed lines of the file:
@@
 F 0 "J3" H 7550 6050 50  0000 C CNN
 F 1 "SPI" V 7650 5750 50  0000 C CNN
-F 2 "Pin_Headers:Pin_Header_Straight_1x05" H 7550 5750 50  0001 C CNN
+F 2 "ESP-RS232:SPI_Header" H 7550 5750 50  0001 C CNN
 F 3 "" H 7550 5750 50  0001 C CNN
 	1    7550 5750

Commit message: Fixed ESP-Sensors board (ht7333 wrong footprint):rev 2
Parts:
- added R4: 10K, Resistors_SMD:R_0805_HandSoldering, symbol R
- J1: footprint Pin_Headers:Pin_Header_Straight_1x05 -> ESP-RS232:Pin_Header_Straight_1x05b
Connections:
- wire segments 86 -> 89
Other:
- note added: "2"
- note added: "2017-04-22"
- note removed: "2017-03-21"
Changed lines of the file:
@@
 EESchema Schematic File Version 2
+LIBS:ESP-Sensors-rescue
 LIBS:power
 LIBS:device
@@
 F 0 "J1" H 7550 3650 50  0000 C CNN
 F 1 "PROG_CONN" V 7650 3350 50  0000 C CNN
-F 2 "Pin_Headers:Pin_Header_Straight_1x05" H 7550 3350 50  0001 C CNN
+F 2 "ESP-RS232:Pin_Header_Straight_1x05b" H 7550 3350 50  0001 C CNN
 F 3 "" H 7550 3350 50  0001 C CNN
 	1    7550 3350
@@
 ESP8266-12E sensor print
 Text Notes 8225 7650 0    60   ~ 0
-2017-03-21
+2017-04-22
 Wire Notes Line
 	8650 800  8650 3000
@@
 Optional power regulator, or feed with 3.3V
 $Comp
-L HT7333 U2
-U 1 1 58E21ABC
-P 9450 2050
-F 0 "U2" H 9725 1825 60  0000 R CNN
-F 1 "HT7333" H 9375 2275 60  0000 C CNN
-F 2 "TO_SOT_Packages_SMD:SOT89-3_Housing_Handsoldering" H 9400 1975 60  0001 C CNN
-F 3 "" H 9400 1975 60  0001 C CNN
-	1    9450 2050
-	1    0    0    -1
-$EndComp
-$Comp
 L CONN_01X02 J5
 U 1 1 58E29D26
@@
 Wire Wire Line
 	2825 2350 2875 2350
+$Comp
+L R R4
+U 1 1 58FB53BE
+P 6800 1850
+F 0 "R4" V 6880 1850 50  0000 C CNN
+F 1 "10K" V 6800 1850 50  0000 C CNN
+F 2 "Resistors_SMD:R_0805_HandSoldering" V 6730 1850 50  0001 C CNN
+F 3 "" H 6800 1850 50  0001 C CNN
+	1    6800 1850
+	-1   0    0    1
+$EndComp
+$Comp
+L GND #PWR09
+U 1 1 58FB53CA
+P 6800 2175
+F 0 "#PWR09" H 6800 1925 50  0001 C CNN
+F 1 "GND" H 6800 2025 50  0000 C CNN
+F 2 "" H 6800 2175 50  0001 C CNN
+F 3 "" H 6800 2175 50  0001 C CNN
+	1    6800 2175
+	1    0    0    -1
+$EndComp
+Text Label 7425 1650 2    60   ~ 0
+GPIO15
+Wire Wire Line
+	6800 1650 7425 1650
+Wire Wire Line
+	6800 2000 6800 2175
+Connection ~ 6800 2175
+Wire Wire Line
+	6800 1650 6800 1700
+Text Notes 10575 7650 0    60   ~ 0
+2
+$Comp
+L HT7333 U2
+U 1 1 590DD42D
+P 9450 2050
+F 0 "U2" H 9725 1825 60  0000 R CNN
+F 1 "HT7333" H 9375 2275 60  0000 C CNN
+F 2 "TO_SOT_Packages_SMD:SOT89-3_Housing_Handsoldering" H 9400 1975 60  0001 C CNN
+F 3 "" H 9400 1975 60  0001 C CNN
+	1    9450 2050
+	1    0    0    -1
+$EndComp
 $EndSCHEMATC
