File: ESP-RS232/ESP-RS232.sch (KiCad schematic (older format))
At the start: 14 parts, among them J1 PROG_CONN, J2 GPIO, J3 CONN_01X05, J4 +5V GND +3.3V, SW1 SW_Push, SW2 SW_Push, U1 ESP-12E

Commit message: First iteration RS232 ESP8266 schematic
Parts:
- removed 10K1: POT, symbol POT
- removed J2: GPIO, symbol CONN_01X12
- removed J3: CONN_01X05, symbol CONN_01X05
- added C? (x5): 100n, symbol C
- added J?: CONN_01X04, symbol CONN_01X04
- added J?: DB9_MALE, symbol DB9_MALE
- added U?: HT7333, symbol HT7333
- added U?: MAX3232, symbol MAX3232
- J4: symbol CONN_01X04 -> CONN_01X04-RESCUE-ESP-RS232
Connections:
- net labels added: CTS, RTS
- net labels removed: ANALOG_IN, CS0, GPIO10, GPIO9, GPIO_BUS, HT7333, MISO, MOSI, SLCK
- wire segments 81 -> 109
- no-connect marks 1 -> 5
Other:
- note added: "Actual pins for RTS/CTS not known yet!"
- note added: "RS-232 to WIFI adapter"
- moved on the sheet: C1, C2, J1, R1, R2, R3, SW1, SW2, U1
