File: 6.0/projects/NodeMCU-Metriful/NodeMCU-Metriful.kicad_sch (KiCad schematic)
At the start: 20 parts, among them CN1 RJ10, CN2 RJ10, CN3 RJ10, J1 Conn_02x04_Odd_Even, J4 Conn_01x03_Female, Q1 BSS138BKW, Q2 NX2301P, U1 NodeMCU_1.0_(ESP-12E), U2 Metriful-1, U3 DS18B20

Commit message: remove doubly-linked connections
Parts:
- U1: footprint (none) -> NodeMCU:NodeMCU_0.1_Axel
Connections:
- net T_enable: no longer Q1.1 (G)
